File: Mykicadedits/base8x/base8x.sch (KiCad schematic (older format))
At the start: 38 parts, among them J1 Conn_02x05_Odd_Even, J2 GS3, J3 Conn_02x14_Counter_Clockwise, J4 GS3, J9 Screw_Terminal_01x08, P3 CONN_01X02, P4 CONN_01X02, U1 ADS1115

Commit message: Updates
Parts:
- removed MK1, MK2: Mounting_Hole_PAD, MountingHole:MountingHole_2.2mm_M2_Pad, symbol base8x-rescue:Mounting_Hole_PAD-Mechanical-base8x-rescue
- removed MK10: Mounting_Hole, MountingHole:MountingHole_4.3mm_M4, symbol base8x-rescue:Mounting_Hole-Mechanical-base8x-rescue
- removed MK11, MK9: Mounting_Hole, MountingHole:MountingHole_6mm, symbol base8x-rescue:Mounting_Hole-Mechanical-base8x-rescue
- D1, D2: footprint myParts:BPW21 -> Resistor_THT:R_Axial_DIN0204_L3.6mm_D1.6mm_P7.62mm_Horizontal
- R1, R2, R3, R4: footprint Resistor_SMD:R_1206_3216Metric -> Resistor_THT:R_Axial_DIN0516_L15.5mm_D5.0mm_P20.32mm_Horizontal
- R5: footprint Resistor_SMD:R_2512_6332Metric -> Resistor_THT:R_Axial_DIN0516_L15.5mm_D5.0mm_P20.32mm_Horizontal
- Resistor1, Resistor_SSR1: footprint Resistor_THT:R_Axial_DIN0617_L17.0mm_D6.0mm_P20.32mm_Horizontal -> Resistor_THT:R_Axial_DIN0516_L15.5mm_D5.0mm_P20.32mm_Horizontal
- TP1, TP2, TP3, TP4, TP5, TP6: footprint myParts:Test_Point_S1751-46R -> TestPoint:TestPoint_Pad_2.5x2.5mm
Connections:
- wire segments 99 -> 94
Changed lines of the file:
@@
 Text Notes 9300 950  0    60   ~ 0
 External Power
-$Comp
-L base8x-rescue:Mounting_Hole_PAD-Mechanical-base8x-rescue MK1
-U 1 1 59C916FE
-P 3300 6100
-F 0 "MK1" H 3400 6151 50  0000 L CNN
-F 1 "Mounting_Hole_PAD" H 3400 6060 50  0000 L CNN
-F 2 "MountingHole:MountingHole_2.2mm_M2_Pad" H 3300 6100 50  0001 C CNN
-F 3 "" H 3300 6100 50  0001 C CNN
-	1    3300 6100
-	1    0    0    -1
-$EndComp
-$Comp
-L base8x-rescue:Mounting_Hole_PAD-Mechanical-base8x-rescue MK2
-U 1 1 59C91760
-P 3300 6450
-F 0 "MK2" H 3400 6501 50  0000 L CNN
-F 1 "Mounting_Hole_PAD" H 3400 6410 50  0000 L CNN
-F 2 "MountingHole:MountingHole_2.2mm_M2_Pad" H 3300 6450 50  0001 C CNN
-F 3 "" H 3300 6450 50  0001 C CNN
-	1    3300 6450
-	1    0    0    -1
-$EndComp
-$Comp
-L power:GND #PWR010
-U 1 1 59C92CEC
-P 3300 6650
-F 0 "#PWR010" H 3300 6400 50  0001 C CNN
-F 1 "GND" H 3300 6500 50  0000 C CNN
-F 2 "" H 3300 6650 50  0000 C CNN
-F 3 "" H 3300 6650 50  0000 C CNN
-	1    3300 6650
-	1    0    0    -1
-$EndComp
 Wire Wire Line
 	2000 6300 2200 6300
@@
 Wire Wire Line
 	9850 1150 9850 1000
-Wire Wire Line
-	3300 6550 3300 6600
-Wire Wire Line
-	3150 6600 3300 6600
-Wire Wire Line
-	3150 6200 3300 6200
-Connection ~ 3300 6600
 Text Label 5050 7450 2    60   ~ 0
 Vin
@@
 Wire Wire Line
 	2350 7100 2350 7150
-Wire Wire Line
-	3150 6200 3150 6600
 $Comp
 L Connector_Generic:Conn_02x05_Odd_Even J1
@@
 F 0 "R4" V 6954 2050 50  0000 C CNN
 F 1 "10K" V 7045 2050 50  0000 C CNN
-F 2 "Resistor_SMD:R_1206_3216Metric" H 7150 2050 50  0001 C CNN
+F 2 "Resistor_THT:R_Axial_DIN0516_L15.5mm_D5.0mm_P20.32mm_Horizontal" H 7150 2050 50  0001 C CNN
 F 3 "" H 7150 2050 50  0001 C CNN
 F 4 "2073607" H 0   0   50  0001 C CNN "farnellCode"
@@
 F 0 "R3" V 7196 2350 50  0000 C CNN
 F 1 "10K" V 7105 2350 50  0000 C CNN
-F 2 "Resistor_SMD:R_1206_3216Metric" H 7000 2350 50  0001 C CNN
+F 2 "Resistor_THT:R_Axial_DIN0516_L15.5mm_D5.0mm_P20.32mm_Horizontal" H 7000 2350 50  0001 C CNN
 F 3 "" H 7000 2350 50  0001 C CNN
 F 4 "2073607" H 0   0   50  0001 C CNN "farnellCode"
@@
 F 0 "D1" V 3700 2900 50  0000 L CNN
 F 1 "BPW21" H 3710 2590 50  0000 C CNN
-F 2 "myParts:BPW21" H 3700 2700 50  0001 C CNN
+F 2 "Resistor_THT:R_Axial_DIN0204_L3.6mm_D1.6mm_P7.62mm_Horizontal" H 3700 2700 50  0001 C CNN
 F 3 "" H 3700 2700 50  0000 C CNN
 F 4 "1045427" H 0   0   50  0001 C CNN "farnellCode"
@@
 F 0 "R1" V 3554 2000 50  0000 C CNN
 F 1 "1.2K" V 3645 2000 50  0000 C CNN
-F 2 "Resistor_SMD:R_1206_3216Metric" H 3750 2000 50  0001 C CNN
+F 2 "Resistor_THT:R_Axial_DIN0516_L15.5mm_D5.0mm_P20.32mm_Horizontal" H 3750 2000 50  0001 C CNN
 F 3 "" H 3750 2000 50  0001 C CNN
 F 4 "2073370" H 0   0   50  0001 C CNN "farnellCode"
@@
 F 0 "D2" V 4250 3550 50  0000 L CNN
 F 1 "BPW21" H 4260 3240 50  0000 C CNN
-F 2 "myParts:BPW21" H 4250 3350 50  0001 C CNN
+F 2 "Resistor_THT:R_Axial_DIN0204_L3.6mm_D1.6mm_P7.62mm_Horizontal" H 4250 3350 50  0001 C CNN
 F 3 "" H 4250 3350 50  0000 C CNN
 F 4 "1045427" H 0   0   50  0001 C CNN "farnellCode"
@@
 F 0 "R2" V 4104 2650 50  0000 C CNN
 F 1 "1.2K" V 4195 2650 50  0000 C CNN
-F 2 "Resistor_SMD:R_1206_3216Metric" H 4300 2650 50  0001 C CNN
+F 2 "Resistor_THT:R_Axial_DIN0516_L15.5mm_D5.0mm_P20.32mm_Horizontal" H 4300 2650 50  0001 C CNN
 F 3 "" H 4300 2650 50  0001 C CNN
 F 4 "2073370" H 0   0   50  0001 C CNN "farnellCode"
@@
 F 0 "TP1" H 5708 6420 50  0000 L CNN
 F 1 "Test_Point" H 5708 6329 50  0000 L CNN
-F 2 "myParts:Test_Point_S1751-46R" H 5850 6300 50  0001 C CNN
+F 2 "TestPoint:TestPoint_Pad_2.5x2.5mm" H 5850 6300 50  0001 C CNN
 F 3 "" H 5850 6300 50  0001 C CNN
 F 4 "2293786" H 0   0   50  0001 C CNN "farnellCode"
@@
 F 0 "TP2" H 4758 1970 50  0000 L CNN
 F 1 "Test_Point" H 4758 1879 50  0000 L CNN
-F 2 "myParts:Test_Point_S1751-46R" H 4900 1850 50  0001 C CNN
+F 2 "TestPoint:TestPoint_Pad_2.5x2.5mm" H 4900 1850 50  0001 C CNN
 F 3 "" H 4900 1850 50  0001 C CNN
 F 4 "2293786" H 0   0   50  0001 C CNN "farnellCode"
@@
 F 0 "R5" H 10420 3096 50  0000 L CNN
 F 1 "1" H 10420 3005 50  0000 L CNN
-F 2 "Resistor_SMD:R_2512_6332Metric" V 10280 3050 50  0001 C CNN
+F 2 "Resistor_THT:R_Axial_DIN0516_L15.5mm_D5.0mm_P20.32mm_Horizontal" V 10280 3050 50  0001 C CNN
 F 3 "" H 10350 3050 50  0001 C CNN
 F 4 "2663692" H 10350 3050 60  0001 C CNN "farnellCode"
@@
 F 0 "TP3" H 4308 2220 50  0000 L CNN
 F 1 "Test_Point" H 4308 2129 50  0000 L CNN
-F 2 "myParts:Test_Point_S1751-46R" H 4450 2100 50  0001 C CNN
+F 2 "TestPoint:TestPoint_Pad_2.5x2.5mm" H 4450 2100 50  0001 C CNN
 F 3 "" H 4450 2100 50  0001 C CNN
 F 4 "2293786" H 0   0   50  0001 C CNN "farnellCode"
@@
 F 0 "TP4" H 5058 2970 50  0000 L CNN
 F 1 "Test_Point" H 5058 2879 50  0000 L CNN
-F 2 "myParts:Test_Point_S1751-46R" H 5200 2850 50  0001 C CNN
+F 2 "TestPoint:TestPoint_Pad_2.5x2.5mm" H 5200 2850 50  0001 C CNN
 F 3 "" H 5200 2850 50  0001 C CNN
 F 4 "2293786" H 0   0   50  0001 C CNN "farnellCode"
@@
 F 0 "TP5" H 5208 1320 50  0000 L CNN
 F 1 "Test_Point" H 5208 1229 50  0000 L CNN
-F 2 "myParts:Test_Point_S1751-46R" H 5350 1200 50  0001 C CNN
+F 2 "TestPoint:TestPoint_Pad_2.5x2.5mm" H 5350 1200 50  0001 C CNN
 F 3 "" H 5350 1200 50  0001 C CNN
 F 4 "2293786" H 0   0   50  0001 C CNN "farnellCode"
@@
 F 0 "TP6" H 10158 3970 50  0000 L CNN
 F 1 "Test_Point" H 10158 3879 50  0000 L CNN
-F 2 "myParts:Test_Point_S1751-46R" H 10300 3850 50  0001 C CNN
+F 2 "TestPoint:TestPoint_Pad_2.5x2.5mm" H 10300 3850 50  0001 C CNN
 F 3 "" H 10300 3850 50  0001 C CNN
 F 4 "2293786" H 0   0   50  0001 C CNN "farnellCode"
@@
 Connection ~ 4250 2150
 Connection ~ 5000 2800
-Wire Wire Line
-	3300 6600 3300 6650
 Wire Wire Line
 	6000 1500 6000 1850
@@
 NoConn ~ 1500 6300
 NoConn ~ 1500 6200
-$Comp
-L base8x-rescue:Mounting_Hole-Mechanical-base8x-rescue MK10
-U 1 1 5AD7C02F
-P 900 1850
-F 0 "MK10" H 1000 1896 50  0000 L CNN
-F 1 "Mounting_Hole" H 1000 1805 50  0000 L CNN
-F 2 "MountingHole:MountingHole_4.3mm_M4" H 900 1850 50  0001 C CNN
-F 3 "" H 900 1850 50  0001 C CNN
-	1    900  1850
-	1    0    0    -1
-$EndComp
-$Comp
-L base8x-rescue:Mounting_Hole-Mechanical-base8x-rescue MK9
-U 1 1 5AD7C3D3
-P 900 1500
-F 0 "MK9" H 1000 1546 50  0000 L CNN
-F 1 "Mounting_Hole" H 1000 1455 50  0000 L CNN
-F 2 "MountingHole:MountingHole_6mm" H 900 1500 50  0001 C CNN
-F 3 "" H 900 1500 50  0001 C CNN
-	1    900  1500
-	1    0    0    -1
-$EndComp
-$Comp
-L base8x-rescue:Mounting_Hole-Mechanical-base8x-rescue MK11
-U 1 1 5AD7C6CB
-P 900 2250
-F 0 "MK11" H 1000 2296 50  0000 L CNN
-F 1 "Mounting_Hole" H 1000 2205 50  0000 L CNN
-F 2 "MountingHole:MountingHole_6mm" H 900 2250 50  0001 C CNN
-F 3 "" H 900 2250 50  0001 C CNN
-	1    900  2250
-	1    0    0    -1
-$EndComp
 Wire Wire Line
 	3050 4000 3525 4000
@@
 F 0 "Resistor1" H 4105 4504 50  0000 R CNN
 F 1 "4.7k" H 4105 4595 50  0000 R CNN
-F 2 "Resistor_THT:R_Axial_DIN0617_L17.0mm_D6.0mm_P20.32mm_Horizontal" V 4105 4550 50  0001 C CNN
+F 2 "Resistor_THT:R_Axial_DIN0516_L15.5mm_D5.0mm_P20.32mm_Horizontal" V 4105 4550 50  0001 C CNN
 F 3 "~" H 4175 4550 50  0001 C CNN
 	1    4175 4550
@@
 F 0 "Resistor_SSR1" H 3580 5229 50  0000 R CNN
 F 1 "?" H 3580 5320 50  0000 R CNN
-F 2 "Resistor_THT:R_Axial_DIN0617_L17.0mm_D6.0mm_P20.32mm_Horizontal" V 3580 5275 50  0001 C CNN
+F 2 "Resistor_THT:R_Axial_DIN0516_L15.5mm_D5.0mm_P20.32mm_Horizontal" V 3580 5275 50  0001 C CNN
 F 3 "~" H 3650 5275 50  0001 C CNN
 	1    3650 5275

Commit message: Big Changes
Parts:
- C1: footprint Capacitor_SMD:C_1206_3216Metric -> Capacitor_THT:CP_Radial_D4.0mm_P1.50mm
Connections:
- net labels added: HELP1, HELP2, HELP3
- wire segments 94 -> 100
- no-connect marks 44 -> 36
Changed lines of the file:
@@
 Text GLabel 10450 1150 1    60   Input ~ 0
 A_V+
-$Comp
-L Connector_Generic:Conn_02x14_Odd_Even J3
-U 1 1 59C14E89
-P 1800 6800
-F 0 "J3" H 1850 7617 50  0000 C CNN
-F 1 "Conn_02x14_Counter_Clockwise" H 1850 7526 50  0001 C CNN
-F 2 "Connector_PinSocket_2.54mm:PinSocket_2x14_P2.54mm_Vertical" H 1800 6800 50  0001 C CNN
-F 3 "" H 1800 6800 50  0001 C CNN
-	1    1800 6800
-	-1   0    0    -1
-$EndComp
 Text Notes 1550 3700 2    60   ~ 0
 COMM_BUS
@@
 F 0 "C1" H 5692 1646 50  0000 L CNN
 F 1 "1uF" H 5692 1555 50  0000 L CNN
-F 2 "Capacitor_SMD:C_1206_3216Metric" H 5600 1600 50  0001 C CNN
+F 2 "Capacitor_THT:CP_Radial_D4.0mm_P1.50mm" H 5600 1600 50  0001 C CNN
 F 3 "" H 5600 1600 50  0001 C CNN
 	1    5600 1600
@@
 	3750 2400 3750 2500
 Wire Wire Line
-	3750 2100 3750 2150
-Wire Wire Line
 	4450 2150 4250 2150
 Connection ~ 3750 2150
@@
 Text GLabel 1250 4550 3    60   Input ~ 0
 A_V_D_LOC
-Text GLabel 850  4550 3    60   Input ~ 0
+Text GLabel 750  4550 3    60   Input ~ 0
 A_V_D_EXT
 Text GLabel 1050 3350 0    60   Input ~ 0
@@
 NoConn ~ 1500 7400
 NoConn ~ 1500 7300
-NoConn ~ 1500 7200
-NoConn ~ 1500 6700
 NoConn ~ 1500 7000
-NoConn ~ 1500 6400
 NoConn ~ 1500 6300
-NoConn ~ 1500 6200
 Wire Wire Line
 	3050 4000 3525 4000
@@
 Wire Wire Line
 	4600 5375 4925 5375
-NoConn ~ 1500 6500
-NoConn ~ 1500 6600
-NoConn ~ 1500 6900
 NoConn ~ 1500 6800
-NoConn ~ 1500 7100
 NoConn ~ 10050 2525
 Wire Wire Line
@@
 Text GLabel 3050 4900 2    50   Input ~ 0
 SCK
+Text GLabel 1500 6400 0    60   Input ~ 0
+SCL
+$Comp
+L power:+5V #PWR0108
+U 1 1 602B69AB
+P 1500 6200
+F 0 "#PWR0108" H 1500 6050 50  0001 C CNN
+F 1 "+5V" H 1500 6340 28  0000 C CNN
+F 2 "" H 1500 6200 50  0000 C CNN
+F 3 "" H 1500 6200 50  0000 C CNN
+	1    1500 6200
+	-1   0    0    -1
+$EndComp
+Text GLabel 1500 6500 0    60   Input ~ 0
+SDA
+Text GLabel 3625 2125 0    50   Input ~ 0
+HELP1
+Wire Wire Line
+	3625 2125 3750 2125
+Wire Wire Line
+	3750 2100 3750 2125
+Connection ~ 3750 2125
+Wire Wire Line
+	3750 2125 3750 2150
+Text GLabel 1500 7200 0    50   Input ~ 0
+HELP1
+Text GLabel 1500 6700 0    50   Input ~ 0
+HELP2
+Text GLabel 800  4475 0    50   Input ~ 0
+HELP2
+Wire Wire Line
+	800  4475 800  4550
+Wire Wire Line
+	750  4550 800  4550
+Connection ~ 800  4550
+Wire Wire Line
+	800  4550 850  4550
+Text GLabel 1500 6900 0    60   Input ~ 0
+A_V_D
+Text GLabel 4300 2800 0    50   Input ~ 0
+HELP3
+Text GLabel 1475 7100 0    50   Input ~ 0
+HELP3
+$Comp
+L Connector_Generic:Conn_02x14_Odd_Even J3
+U 1 1 59C14E89
+P 1800 6800
+F 0 "J3" H 1850 7617 50  0000 C CNN
+F 1 "Conn_02x14_Counter_Clockwise" H 1850 7526 50  0001 C CNN
+F 2 "Connector_PinSocket_2.54mm:PinSocket_2x14_P2.54mm_Vertical" H 1800 6800 50  0001 C CNN
+F 3 "" H 1800 6800 50  0001 C CNN
+	1    1800 6800
+	-1   0    0    -1
+$EndComp
+Wire Wire Line
+	1475 7100 1500 7100
+Text GLabel 1500 6600 0    50   Input ~ 0
+HELP3
 $EndSCHEMATC
