File: Mykicadedits/base8x/base8x.kicad_pcb (KiCad board)
At the start: 4 copper layers, 25 parts, among them J1 Conn_02x05_Odd_Even, J2 GS3, J3 Conn_02x14_Counter_Clockwise, J4 GS3, J9 Screw_Terminal_01x08, P3 CONN_01X02, P4 CONN_01X02, U1 ADS1115

Commit message: Updates
Parts:
- added D1: BPW21, Resistor_THT:R_Axial_DIN0204_L3.6mm_D1.6mm_P7.62mm_Horizontal, F.Cu at (-176.7, 10.2)
- added D2: BPW21, Resistor_THT:R_Axial_DIN0204_L3.6mm_D1.6mm_P7.62mm_Horizontal, F.Cu at (-176.7, 13.4)
- added TP1: Test_Point, TestPoint:TestPoint_Pad_2.5x2.5mm, F.Cu at (-42.9, -27.0)
- added TP2: Test_Point, TestPoint:TestPoint_Pad_2.5x2.5mm, F.Cu at (-63.1, -25.8)
- added TP3: Test_Point, TestPoint:TestPoint_Pad_2.5x2.5mm, F.Cu at (-63.1, -21.3)
- added TP4: Test_Point, TestPoint:TestPoint_Pad_2.5x2.5mm, F.Cu at (-58.6, -25.8)
- added TP5: Test_Point, TestPoint:TestPoint_Pad_2.5x2.5mm, F.Cu at (-58.6, -21.3)
- added TP6: Test_Point, TestPoint:TestPoint_Pad_2.5x2.5mm, F.Cu at (-38.4, -27.0)
- R1, R2, R3, R4: footprint Resistor_SMD:R_1206_3216Metric -> Resistor_THT:R_Axial_DIN0516_L15.5mm_D5.0mm_P20.32mm_Horizontal
- R5: footprint Resistor_SMD:R_2512_6332Metric -> Resistor_THT:R_Axial_DIN0516_L15.5mm_D5.0mm_P20.32mm_Horizontal
- Resistor1, Resistor_SSR1: footprint Resistor_THT:R_Axial_DIN0617_L17.0mm_D6.0mm_P20.32mm_Horizontal -> Resistor_THT:R_Axial_DIN0516_L15.5mm_D5.0mm_P20.32mm_Horizontal
- moved P4 406.3 mm to (-242.1, 24.4), turned to 270 degrees
- moved R1 363.4 mm to (-226.7, 137.1)
- moved J3 345.2 mm to (-255.4, 57.0)
- moved SSR-Ithink1 312.3 mm to (-184.5, 75.6)
- moved J9 310.9 mm to (-255.5, 31.5)
- moved R2 281.3 mm to (-136.4, 144.3)
- moved Raspberry_header1 280.8 mm to (-244.9, 57.0)
- moved C1 277.2 mm to (-89.6, 31.8)
- moved J1 277.2 mm to (-154.4, 41.2)
- moved J2 277.2 mm to (-122.1, 93.3)
- moved J4 277.2 mm to (-127.3, 100.5)
- moved JP2 277.2 mm to (-90.3, 28.2)
- moved JP3 277.2 mm to (-168.8, -25.0)
- moved JP4 277.2 mm to (-85.9, 28.2)
- moved JP5 277.2 mm to (-207.7, -15.8)
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Routing:
- net A_V-: track 0.00 -> 87.4 mm
- net A_V+: track 0.00 -> 85.3 mm
- net A_I+: track 0.00 -> 83.8 mm
- net A_I-: track 0.00 -> 81.8 mm
- net GND: track 0.00 -> 37.2 mm
- net MISO: track 0.00 -> 21.3 mm
- net SCL: track 0.00 -> 12.7 mm
- net SDA: track 0.00 -> 12.7 mm
- net MOSI: track 0.00 -> 12.7 mm
- net +3V3: track 0.00 -> 11.6 mm
- net SCK: track 0.00 -> 11.2 mm
- net +5V: track 0.00 -> 8.05 mm

Commit message: Big Changes
Parts:
- C1: footprint Capacitor_SMD:C_1206_3216Metric -> Capacitor_THT:CP_Radial_D4.0mm_P1.50mm
- JP6: moved to B.Cu
- moved TP4 270.8 mm to (-308.4, 78.7)
- moved Resistor1 262.7 mm to (-302.5, 36.1)
- moved TP1 238.5 mm to (-251.8, 88.0)
- moved JP4 231.3 mm to (-312.4, 75.2), turned to 90 degrees
- moved TP5 230.7 mm to (-269.1, 73.2)
- moved TP2 228.4 mm to (-270.9, 68.9)
- moved TP3 222.5 mm to (-266.5, 68.9)
- moved TP6 221.2 mm to (-249.3, 39.5)
- moved JP2 216.2 mm to (-305.7, 46.6)
- moved C1 195.0 mm to (-283.7, 51.0)
- moved R3 182.0 mm to (-276.0, 76.6), turned to 90 degrees
- moved Temp_sensor1 179.3 mm to (-282.3, 41.3)
- moved R2 178.0 mm to (-301.1, 76.8), turned to 90 degrees
- moved U1 174.0 mm to (-268.8, 64.4)
- moved R5 173.3 mm to (-269.3, 44.8)
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Connections:
- J3 pad 10: Net-(J3-Pad10) -> HELP3
- J3 pad 12: Net-(J3-Pad12) -> A_V_D_EXT
- J3 pad 16: Net-(J3-Pad16) -> A_V_D
- J3 pad 2: Net-(J3-Pad2) -> +5V
- J3 pad 20: Net-(J3-Pad20) -> HELP3
- J3 pad 22: Net-(J3-Pad22) -> HELP1
- J3 pad 6: Net-(J3-Pad6) -> SCL
- J3 pad 8: Net-(J3-Pad8) -> SDA
- JP2 pad 1: Net-(JP2-Pad1) -> HELP1
- JP4 pad 1: Net-(JP4-Pad1) -> HELP3
- R1 pad 1: Net-(JP2-Pad1) -> HELP1
- R2 pad 1: Net-(JP4-Pad1) -> HELP3
- TP3 pad 1: Net-(JP2-Pad1) -> HELP1
- TP4 pad 1: Net-(JP4-Pad1) -> HELP3
- U1 pad 6: Net-(JP2-Pad1) -> HELP1
- U1 pad 7: Net-(JP4-Pad1) -> HELP3
Routing:
- net GND: track 37.2 -> 389.6 mm
- net A_I-: track 81.8 -> 326.3 mm
- net HELP1: track 0.00 -> 237.9 mm
- net A_V-: track 87.4 -> 290.2 mm
- net A_V+: track 85.3 -> 281.2 mm
- net A_I+: track 83.8 -> 269.3 mm
- net SCK: track 11.2 -> 147.8 mm
- net MOSI: track 12.7 -> 141.1 mm
- net +5V: track 8.05 -> 133.1 mm
- net MISO: track 21.3 -> 144.8 mm
- net ~A_CS: track 0.00 -> 93.2 mm
- net HELP3: track 0.00 -> 90.7 mm
- net SCL: track 12.7 -> 92.0 mm
- net CLK0: track 0.00 -> 77.9 mm
- net A_V_D_EXT: track 0.00 -> 74.3 mm
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Other:
- board outline added: 260.8 x 212.2 mm

Commit message: Finishing Touches
Other:
- board size 260.8 x 212.2 mm -> 191 x 106.2 mm
