File: KiCad2.0/solar_mux/solar_mux.sch (KiCad schematic (older format))
At the start: 35 parts, among them J1 Conn_01x14, J2 Conn_02x06_Odd_Even, J3 Conn_02x06_Odd_Even, U1 ASSR-1611, U10 ASSR-1611, U11 ASSR-1611, U12 ASSR-1611, U13 ASSR-1611, U14 ASSR-1611, U15 ASSR-1611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

Commit message: major rebuild
Parts:
- removed help1: Conn_01x04, Connector_PinHeader_2.00mm:PinHeader_1x04_P2.00mm_Vertical, symbol Connector_Generic:Conn_01x04
- added J4: Conn_01x14, Connector_PinHeader_2.54mm:PinHeader_1x14_P2.54mm_Vertical, symbol Connector_Generic:Conn_01x14
- added JP6: Jumper_NC_Small, Jumper:SolderJumper-2_P1.3mm_Open_RoundedPad1.0x1.5mm, symbol Device:Jumper_NC_Small
- added L1: grey@mutovis.com, logo:text, symbol solar_mux-rescue:logo_text-logo
- C1: footprint Capacitor_THT:CP_Radial_D8.0mm_P2.50mm -> Capacitor_SMD:C_1206_3216Metric_Pad1.42x1.75mm_HandSolder
- J2: footprint Connector_PinHeader_2.54mm:PinHeader_2x06_P2.54mm_Vertical -> myParts:ESQ-106-44-G-D-004
- J3: footprint Connector_PinHeader_2.54mm:PinHeader_2x06_P2.54mm_Vertical -> myParts:ESQ-106-44-G-D
- R1, R2, R3, R4: footprint Resistor_THT:R_Axial_DIN0309_L9.0mm_D3.2mm_P15.24mm_Horizontal -> Resistor_SMD:R_1206_3216Metric_Pad1.42x1.75mm_HandSolder
- TP1: footprint TestPoint:TestPoint_Pad_2.5x2.5mm -> myParts:Test_Point_S1751-46R
- U1, U10, U11, U12, U13, U14, U15, U16, U17, U2, U20, U21, U3, U4, U5, U6, U7: symbol solar_mux_1-rescue:ASSR-1611-myParts-solar_mux-rescue -> solar_mux-rescue:ASSR-1611-myParts
Connections:
- net labels added: P7, P8
- wire segments 157 -> 163
- no-connect marks 31 -> 29
Other:
- note added: "RIGHT SIDE BUS CONNECTIONS"
