File: KiCad2.0/solar_mux/Solar_Multiplexer.sch (KiCad schematic (older format))
At the start: 37 parts, among them J1 Conn_01x14, J2 Conn_02x06_Odd_Even, J3 Conn_02x06_Odd_Even, J4 Conn_01x14, U1 ASSR-1611, U10 ASSR-1611, U11 ASSR-1611, U12 ASSR-1611, U13 ASSR-1611, U14 ASSR-1611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

Commit message: big edits
Parts:
- removed J4: Conn_01x14, Connector_PinHeader_2.54mm:PinHeader_1x14_P2.54mm_Vertical, symbol Connector_Generic:Conn_01x14
- removed JP6: Jumper_NC_Small, Jumper:SolderJumper-2_P1.3mm_Open_RoundedPad1.0x1.5mm, symbol Device:Jumper_NC_Small
- removed L1: grey@mutovis.com, logo:text, symbol solar_mux-rescue:logo_text-logo
- C1: footprint Capacitor_SMD:C_1206_3216Metric_Pad1.42x1.75mm_HandSolder -> Capacitor_THT:CP_Radial_D8.0mm_P2.50mm
- J2: footprint myParts:ESQ-106-44-G-D-004 -> Connector_PinHeader_2.54mm:PinHeader_2x06_P2.54mm_Vertical
- J3: footprint myParts:ESQ-106-44-G-D -> Connector_PinHeader_2.54mm:PinHeader_2x06_P2.54mm_Vertical
- R1, R2, R3, R4: footprint Resistor_SMD:R_1206_3216Metric_Pad1.42x1.75mm_HandSolder -> Resistor_THT:R_Axial_DIN0309_L9.0mm_D3.2mm_P15.24mm_Horizontal
- TP1: footprint myParts:Test_Point_S1751-46R -> TestPoint:TestPoint_Pad_2.5x2.5mm
- U1, U10, U11, U12, U13, U14, U15, U16, U17, U2, U20, U21, U3, U4, U5, U6, U7: symbol solar_mux-rescue:ASSR-1611-myParts -> solar_mux_1-rescue:ASSR-1611-myParts-solar_mux-rescue
Connections:
- net labels removed: P7, P8
- wire segments 163 -> 153
- no-connect marks 29 -> 31
Other:
- note removed: "RIGHT SIDE BUS CONNECTIONS"
