File: KiCad2.0/solar_mux/Solar_Multiplexer.kicad_pcb (KiCad board)
At the start: 2 copper layers, 229.4 x 213.5 mm, 34 parts, among them J1 Conn_01x14, J2 Conn_02x06_Odd_Even, J3 Conn_02x06_Odd_Even, U1 ASSR-1611, U10 ASSR-1611, U11 ASSR-1611, U12 ASSR-1611, U13 ASSR-1611, U14 ASSR-1611, U15 ASSR-1611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

Commit message: Final Edits
Parts:
- added REF**: MountingHole_2.2mm_M2, MountingHole:MountingHole_2.2mm_M2, F.Cu at (-310.0, 253.0)
- added REF**: MountingHole_2.2mm_M2, MountingHole:MountingHole_2.2mm_M2, F.Cu at (-200.0, 254.0)
- added REF**: MountingHole_2.2mm_M2, MountingHole:MountingHole_2.2mm_M2, F.Cu at (-200.0, 75.0)
- added REF**: MountingHole_2.2mm_M2, MountingHole:MountingHole_2.2mm_M2, F.Cu at (-310.0, 75.0)
Other:
- board size 229.4 x 213.5 mm -> 205 x 190 mm
